File: hardware/ADXL337 Breakout.brd (EAGLE design)
At the start: 17.8 x 17.8 mm, 13 parts, among them U1 ADXL337

Commit message: v10 ready for review
Parts:
- U1: device SparkFun-Sensors:ADXL337 -> SparkFun-Sensors:LFCSP_LQ-16
- moved LOGO2 1.02 mm to (16.3, 8.89)
Other:
- board text added: "3.3V"
- board text added: "v10"
- board text added: "±3g"
- board text removed: "VCC"
- board text removed: "v01"
Changed lines of the file:
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@@
 <layer number="29" name="tStop" color="7" fill="3" visible="no" active="yes"/>
 <layer number="30" name="bStop" color="7" fill="6" visible="no" active="yes"/>
-<layer number="31" name="tCream" color="7" fill="4" visible="yes" active="yes"/>
+<layer number="31" name="tCream" color="7" fill="4" visible="no" active="yes"/>
 <layer number="32" name="bCream" color="7" fill="5" visible="no" active="yes"/>
 <layer number="33" name="tFinish" color="6" fill="3" visible="no" active="yes"/>
@@
 <text x="5.588" y="15.24" size="1.27" layer="21" font="vector" ratio="15" rot="R90">Y</text>
 <text x="3.048" y="2.921" size="1.27" layer="21" font="vector" ratio="15" rot="R90">GND</text>
-<text x="5.715" y="2.921" size="1.27" layer="21" font="vector" ratio="15" rot="R90">VCC</text>
+<text x="5.715" y="2.921" size="1.27" layer="21" font="vector" ratio="15" rot="R90">3.3V</text>
 <text x="8.255" y="2.921" size="1.27" layer="21" font="vector" ratio="15" rot="R90">X</text>
 <text x="10.668" y="2.921" size="1.27" layer="21" font="vector" ratio="15" rot="R90">Y</text>
@@
 <text x="15.875" y="2.921" size="1.27" layer="21" font="vector" ratio="15" rot="R90">ST</text>
 <text x="17.145" y="4.826" size="1.27" layer="21" font="vector" ratio="15" rot="R90">ADXL337</text>
-<text x="1.778" y="16.764" size="1.27" layer="16" font="vector" ratio="15" rot="SMR270">v01</text>
-<text x="12.319" y="12.827" size="1.27" layer="22" font="vector" ratio="15" rot="SMR270">ADXL337</text>
+<text x="1.778" y="16.764" size="1.27" layer="16" font="vector" ratio="15" rot="SMR270">v10</text>
+<text x="12.192" y="12.827" size="1.27" layer="22" font="vector" ratio="15" rot="SMR270">ADXL337</text>
 <text x="-1.27" y="-19.05" size="1.27" layer="25" font="vector" ratio="15">Jordan McConnell</text>
+<text x="14.224" y="10.414" size="1.27" layer="22" font="vector" ratio="15" rot="SMR270">±3g</text>
 </plain>
 <attributes>
@@
 <elements>
 <element name="FRAME1" library="SparkFun-Aesthetics" package="CREATIVE_COMMONS" value="FRAME-LETTER" x="-11.43" y="-16.51"/>
-<element name="U1" library="SparkFun-Sensors" package="ADXL337" value="ADXL337" x="8.89" y="10.16"/>
+<element name="U1" library="SparkFun-Sensors" package="LFCSP_LQ-16" value="ADXL337" x="8.89" y="10.16"/>
 <element name="JP1" library="SparkFun-Connectors" package="1X06" value="" x="2.54" y="1.27"/>
 <element name="C1" library="SparkFun-Capacitors" package="0603-CAP" value="10nF" x="8.89" y="6.35">
@@
 <element name="STANDOFF1" library="SparkFun-Electromechanical" package="STAND-OFF" value="STAND-OFF" x="15.24" y="15.24"/>
 <element name="LOGO1" library="SparkFun-Aesthetics" package="SFE_LOGO_FLAME_.1" value="SFE_LOGO_FLAME.1_INCH" x="12.192" y="14.351" rot="R90"/>
-<element name="LOGO2" library="SparkFun-Aesthetics" package="OSHW-LOGO-S" value="OSHW-LOGOS" x="15.24" y="8.89" rot="MR270"/>
+<element name="LOGO2" library="SparkFun-Aesthetics" package="OSHW-LOGO-S" value="OSHW-LOGOS" x="16.256" y="8.89" rot="MR270"/>
 <element name="LOGO3" library="SparkFun-Aesthetics" package="SFE_LOGO_NAME_FLAME_.1" value="SFE_LOGO_NAME_FLAME.1_INCH" x="10.414" y="14.732" rot="MR270"/>
 </elements>
