File: hardware/ADXL337 Breakout.sch (EAGLE design)
At the start: 13 parts, among them U1 ADXL337

Commit message: v10 ready for review
Other:
- note added: "v10"
- note removed: "v01"
Changed lines of the file:
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@@
 <plain>
 <text x="149.86" y="7.62" size="2.54" layer="94">Jordan McConnell</text>
-<text x="238.76" y="7.62" size="2.54" layer="94">v01</text>
+<text x="238.76" y="7.62" size="2.54" layer="94">v10</text>
 </plain>
 <instances>
